File: _autosave-Discriminator.kicad_sch (KiCad schematic)
At the start: 74 parts, among them J1 Conn_01x05_Socket, J2 Conn_01x05_Socket, J3 Conn_Coaxial, J4 Conn_01x05_Socket, J5 Conn_01x05_Socket, J6 Conn_01x05_Socket, J7 Conn_01x05_Socket, J8 Conn_01x05_Socket, U1 PSA4-5043+, U2 PGA-103+, U5 DAC60501-0x49

Commit message: added mcu section, added test points to CTD
Parts:
- gave numbers to parts that had none: 3
Changed lines of the file:
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@@
 		(dnp no)
 		(fields_autoplaced yes)
-		(property "Reference" "R?"
+		(property "Reference" "R14"
 			(at 105.41 161.29 90)
 			(effects
@@
 			(project "Discriminator"
 				(path "/98ea3513-a87d-444b-a2da-a8556e3bcd2d"
-					(reference "R?")
+					(reference "R14")
 					(unit 1)
 				)
@@
 		(dnp no)
 		(fields_autoplaced yes)
-		(property "Reference" "R?"
+		(property "Reference" "R13"
 			(at 104.14 170.1799 0)
 			(effects
@@
 			(project "Discriminator"
 				(path "/98ea3513-a87d-444b-a2da-a8556e3bcd2d"
-					(reference "R?")
+					(reference "R13")
 					(unit 1)
 				)
@@
 		(dnp no)
 		(fields_autoplaced yes)
-		(property "Reference" "R?"
+		(property "Reference" "R5"
 			(at 97.79 162.2312 90)
 			(effects
@@
 			(project "Discriminator"
 				(path "/98ea3513-a87d-444b-a2da-a8556e3bcd2d"
-					(reference "R?")
+					(reference "R5")
 					(unit 1)
 				)

Commit message: Misc changes
Parts:
- L1, L3: value L -> 100nh
- R6: value 2k -> 4.7k
Other:
- note added: "Input"
- note added: "https://www.analog.com/media/en/technical-documentation/data-sheets/6752fc.pdf"
- note added: "https://www.minicircuits.com/pdfs/PGA-103+.pdf"
- note added: "https://www.minicircuits.com/pdfs/PSA4-5043+.pdf?srsltid=AfmBOopbdupT7FMYAgyD6TNCni1rLVrMsZ3Wdixk_LjpdAJLGQMF5Q6_"
- moved on the sheet: D_Life3.3, D_Life5, J1, R2, R6, TP4, TP7, TP8
