File: Compute/Discriminator.kicad_sch (KiCad schematic)
At the start: 74 parts, among them J1 Conn_01x05_Socket, J2 Conn_01x05_Socket, J3 Conn_Coaxial, J4 Conn_01x05_Socket, J5 Conn_01x05_Socket, J6 Conn_01x05_Socket, J7 Conn_01x05_Socket, J8 Conn_01x05_Socket, U1 PSA4-5043+, U2 PGA-103+, U5 DAC60501-0x49

Commit message: Complete separation of CTD & Compute, completed Compute BOM, fixed issues
Parts:
- removed C1, C2, C4, C8: 0.01uf, Capacitor_SMD:C_0402_1005Metric, symbol Device:C
- removed C10: 0.33uf, Capacitor_SMD:C_0603_1608Metric, symbol Device:C
- removed C11, C6: 10uf, Capacitor_SMD:C_0805_2012Metric, symbol Device:C
- removed C12, C14, C5: 0.1uf, Capacitor_SMD:C_0603_1608Metric, symbol Device:C
- removed C13, C15: 1uf, Capacitor_SMD:C_0603_1608Metric, symbol Device:C
- removed C3: 100pf, Capacitor_SMD:C_0402_1005Metric, symbol Device:C
- removed C7: 330pf, Capacitor_SMD:C_0603_1608Metric, symbol Device:C
- removed C9: 330pf, Capacitor_SMD:C_0402_1005Metric, symbol Device:C
- removed D_Life3.3, D_Life5: LED, LED_SMD:LED_0603_1608Metric, symbol Device:LED
- removed J1: Conn_01x05_Socket, Connector_JST:JST_XH_B5B-XH-A_1x05_P2.50mm_Vertical, symbol Connector:Conn_01x05_Socket
- removed J3: Conn_Coaxial, Connector_Coaxial:SMA_Samtec_SMA-J-P-H-ST-EM1_EdgeMount, symbol Connector:Conn_Coaxial
- removed L1, L3: 100nh, TCCH+:GU1604_MNC, symbol Device:L
- removed L2: 620nH, Inductor_SMD:L_0603_1608Metric, symbol Device:L
- removed R1: 150, Resistor_SMD:R_0603_1608Metric, symbol Device:R
- removed R2: 2k, Capacitor_SMD:C_0603_1608Metric, symbol Device:R
- removed R6: 4.7k, Capacitor_SMD:C_0603_1608Metric, symbol Device:R
- removed R_Hyst1: 80k, Resistor_SMD:R_0603_1608Metric, symbol Device:R
- removed R_a1: 5.6k, Resistor_SMD:R_0603_1608Metric, symbol Device:R
- removed R_b1: 1k, Resistor_SMD:R_0603_1608Metric, symbol Device:R
- removed R_s1, Rterm1: 50, Resistor_SMD:R_0402_1005Metric, symbol Device:R
- removed TP1, TP2, TP3, TP4, TP5, TP6, TP7, TP8, TP9: TestPoint, TestPoint:TestPoint_Pad_1.5x1.5mm, symbol Connector:TestPoint
- removed U1: PSA4-5043+, PSA4-5043+:MMM1362_MNC, symbol RF_Amplifier:PGA-103
- removed U2: PGA-103+, Package_TO_SOT_SMD:SOT-89-3, symbol RF_Amplifier:PGA-103
- removed U_Comparator1: LTC6752xSC6-1, Package_TO_SOT_SMD:SOT-363_SC-70-6, symbol Comparator:LTC6752xSC6-1
- 3386F-1-201LF1: renamed from RM-065-201; footprint Potentiometer_THT:Potentiometer_Runtron_RM-065_Vertical -> Potentiometer_THT:Potentiometer_Bourns_3386F_Vertical
- R10, R11, R12, R7, R8, R9: footprint Capacitor_SMD:C_0603_1608Metric -> Resistor_SMD:R_0603_1608Metric
Other:
- note removed: "Input"
- note removed: "https://www.analog.com/media/en/technical-documentation/data-sheets/6752fc.pdf"
- note removed: "https://www.minicircuits.com/pdfs/PGA-103+.pdf"
- note removed: "https://www.minicircuits.com/pdfs/PSA4-5043+.pdf?srsltid=AfmBOopbdupT7FMYAgyD6TNCni1rLVrMsZ3Wdixk_LjpdAJLGQMF5Q6_"
- moved on the sheet: 3386F-1-201LF1, C16, C17, C18, C19, C20, J2, J4, J5, J6, J7, J8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
