File: CTD/Discriminator.kicad_sch (KiCad schematic)
At the start: 34 parts, among them J3 Conn_Coaxial, U1 PSA4-5043+, U2 PGA-103+

Commit message: tweaks and bug fixes
Parts:
- added D_Life3.3, D_Life5: LED, LED_SMD:LED_0603_1608Metric, symbol Device:LED
- added J1: Conn_01x05_Socket, Connector_JST:JST_XH_B5B-XH-A_1x05_P2.50mm_Vertical, symbol Connector:Conn_01x05_Socket
- added R2: 2k, Resistor_SMD:R_0603_1608Metric, symbol Device:R
- added R6: 4.7k, Resistor_SMD:R_0603_1608Metric, symbol Device:R
- added TP4, TP7, TP8: TestPoint, TestPoint:TestPoint_Pad_1.0x1.0mm, symbol Connector:TestPoint
- TP1, TP2, TP3, TP5, TP6, TP9: footprint TestPoint:TestPoint_Pad_1.5x1.5mm -> TestPoint:TestPoint_Pad_1.0x1.0mm; now fitted
Connections:
- net +3.3V: now also D_Life3.3.2 (A), J1.4 (Pin_4), TP7.1
- net +5V: now also D_Life5.2 (A), J1.5 (Pin_5), TP4.1
- net GND: now also J1.2 (Pin_2), R2.2, R6.2, TP8.1
- net Pulse: now also J1.1 (Pin_1)
- net V_threshold: now also J1.3 (Pin_3)
- new net: D_Life3.3.1 (K), R2.1
- new net: D_Life5.1 (K), R6.1
