File: Single-Board/Discriminator.kicad_pcb (KiCad board)
At the start: 4 copper layers, 60 x 100.9 mm, 78 parts, among them J1 Conn_01x05_Socket, J2 Conn_01x05_Socket, J3 Conn_Coaxial, J4 Conn_01x05_Socket, J5 Conn_01x05_Socket, J6 Conn_01x05_Socket, J7 Conn_01x05_Socket, J8 Conn_01x05_Socket, U1 PSA4-5043+, U2 PGA-103+, U5 DAC60501-0x49

Commit message: separate CTD & compute. Add CTD BOM
Parts:
- added R13: 1k, Resistor_SMD:R_0603_1608Metric, F.Cu at (125.5, 113.3)
- added R14: 1k, Resistor_SMD:R_0603_1608Metric, F.Cu at (125.5, 120.3)
- added R5: 5.6k, Resistor_SMD:R_0603_1608Metric, F.Cu at (125.5, 116.8)
- added RM-065-201: 200ohms, Potentiometer_THT:Potentiometer_Runtron_RM-065_Vertical, F.Cu at (172.5, 124.5)
- R6: value 2k -> 4.7k
Connections:
- J8 pad 3: /V_r -> Net-(J8-Pin_3)
Routing:
- net Net-(R14-Pad1): track 0.00 -> 48.5 mm
- net /V_r: track 150.7 -> 138.4 mm
- net GNDA: track 1.65 -> 13.7 mm, vias 16 -> 19
- net Net-(R13-Pad2): track 0.00 -> 7.32 mm
- net +3.3VA: track 189.2 -> 194.6 mm
- net Net-(J8-Pin_3): track 0.00 -> 4.95 mm
- net GND: vias 160 -> 155
Other:
- board text added: "J8 V_th"

Commit message: tweaks and bug fixes
Parts:
- 3386F-1-201LF1: renamed from RM-065-201; footprint Potentiometer_THT:Potentiometer_Runtron_RM-065_Vertical -> Potentiometer_THT:Potentiometer_Bourns_3386F_Vertical
- L1, L3: value L -> 100nh
- R10, R11, R12, R2, R6, R7, R8, R9: footprint Capacitor_SMD:C_0603_1608Metric -> Resistor_SMD:R_0603_1608Metric
- moved 3386F-1-201LF1 0.25 mm to (172.2, 124.5), turned to 0 degrees
Routing:
- net Net-(3386F-1-201LF1-Pad1): track 48.5 -> 50.1 mm
